File: aux_port.kicad_sch (KiCad schematic)
At the start: 5 parts, among them J1 USB_C

Commit message: add first round of hits on lcsc
Parts:
- D25: LCSC# (none) -> C503417
- J1: LCSC# (none) -> C2927039
- R44: LCSC# (none) -> C105873
