File: bank8_configuration.kicad_sch (KiCad schematic)
At the start: 19 parts, among them IC1 ECP5-BGA256, U7 W25Q32JVSS

Commit message: add first round of hits on lcsc
Parts:
- C35: LCSC# (none) -> C100072
- R102, R109, R13, R6: LCSC# (none) -> C105873
- R110: LCSC# (none) -> C60489
- R5: LCSC# (none) -> C163447
- U7: LCSC# (none) -> C179173
