File: clock_misc.kicad_sch (KiCad schematic)
At the start: 18 parts, among them J11 SPRING_CONTACT, J12 SPRING_CONTACT, J13 SPRING_CONTACT, J14 SPRING_CONTACT, J15 SPRING_CONTACT, J16 SPRING_CONTACT, Y1 Osc60MHz

Commit message: add first round of hits on lcsc
Parts:
- C10: LCSC# (none) -> C100072
