File: control_port.kicad_sch (KiCad schematic)
At the start: 15 parts, among them J2 USB_C, U16 PI3USB102G

Commit message: add first round of hits on lcsc
Parts:
- C25, C47: LCSC# (none) -> C13533
- C61: LCSC# (none) -> C100072
- C62: LCSC# (none) -> C14442
- D23: LCSC# (none) -> C503417
- J2: LCSC# (none) -> C2927039
- R15: LCSC# (none) -> C60489
- R34, R35, R46: LCSC# (none) -> C105873
- R55, R56: LCSC# (none) -> C137838
- U16: LCSC# (none) -> C155356
