File: expansion.kicad_sch (KiCad schematic)
At the start: 8 parts, among them J5 MEZZANINE, J7 PMOD_A, J8 PMOD_B

Commit message: add first round of hits on lcsc
Parts:
- C74: LCSC# (none) -> C318573
- J5: LCSC# (none) -> C5409782
- RN1, RN2, RN3, RN4: LCSC# (none) -> C125323
