File: indicators_buttons.kicad_sch (KiCad schematic)
At the start: 43 parts, among them SW1 BTN_PROGRAM, SW2 BTN_RESET, SW3 BTN_USER

Commit message: add first round of hits on lcsc
Parts:
- C76, C78: LCSC# (none) -> C318573
- D10, D14: LCSC# (none) -> C389522
- D3: LCSC# (none) -> C375450
- D4: LCSC# (none) -> C375445
- D5: LCSC# (none) -> C205443
- D6: LCSC# (none) -> C193191
- R10, R30, R31, R8, R9: LCSC# (none) -> C163447
- R101: LCSC# (none) -> C2076955
- R106, R29: LCSC# (none) -> C60489
- R11, R7: LCSC# (none) -> C105873
- R26, R27, R28: LCSC# (none) -> C105637
- SW1, SW2, SW3: LCSC# (none) -> C692468
