File: target_port.kicad_sch (KiCad schematic)
At the start: 10 parts, among them J3 USB_A, J4 USB_C

Commit message: add first round of hits on lcsc
Parts:
- D24, D26: LCSC# (none) -> C503417
- J3: LCSC# (none) -> C42411
- J4: LCSC# (none) -> C2927039
- R45: LCSC# (none) -> C105873
- R57, R58: LCSC# (none) -> C105637
