File: usb_phy.kicad_sch (KiCad schematic)
At the start: 14 parts, among them U8 USB3343-CP

Commit message: add first round of hits on lcsc
Parts:
- C36, C37: LCSC# (none) -> C318573
- C38, C39: LCSC# (none) -> C100072
- FL3: LCSC# (none) -> C882594
- R16: LCSC# (none) -> C2076955
- R17: LCSC# (none) -> C137902
- R22: LCSC# (none) -> C60489
- RN5, RN6, RN7: LCSC# (none) -> C106231
- U8: LCSC# (none) -> C633347
